Commit message: 更新仿真

File: src/vendor_robot_description/urdf/g4.model.xacro (robot description, xacro)
@@ -399,3 +399,7 @@
       velocity="6.28" />
   </joint>
+  <xacro:include filename="gripper.xacro"/>
+  <xacro:wsg_50_gripper prefix="${prefix}" parent="${prefix}Link6">
+    <origin xyz="0 0 0.1" rpy="0 0 0"/>
+  </xacro:wsg_50_gripper>
 </robot>

File: src/vendor_robot_moveit_config/config/G4.srdf.xacro (robot description, xacro)
@@ -11,4 +11,12 @@
     <joint name="${prefix}joint6"/>
   </group>
+  <!-- The right guide is a URDF mimic joint, so only the left coordinate is planned. -->
+  <group name="gripper">
+    <joint name="${prefix}gripper_left_joint"/>
+  </group>
+  <end_effector name="${prefix}gripper"
+                parent_link="${prefix}Link6"
+                group="gripper"
+                parent_group="arm"/>
   <group_state name="pose1" group="arm">
     <joint name="${prefix}joint1" value="0"/>
@@ -18,4 +26,10 @@
     <joint name="${prefix}joint5" value="0"/>
     <joint name="${prefix}joint6" value="0"/>
+  </group_state>
+  <group_state name="open" group="gripper">
+    <joint name="${prefix}gripper_left_joint" value="-0.055"/>
+  </group_state>
+  <group_state name="closed" group="gripper">
+    <joint name="${prefix}gripper_left_joint" value="-0.0027"/>
   </group_state>
   <disable_collisions link1="${prefix}Link1" link2="${prefix}Link2" reason="Adjacent"/>
@@ -30,3 +44,8 @@
   <disable_collisions link1="${prefix}Link4" link2="${prefix}Link6" reason="Never"/>
   <disable_collisions link1="${prefix}Link5" link2="${prefix}Link6" reason="Adjacent"/>
+  <disable_collisions link1="${prefix}Link6" link2="${prefix}gripper_base_link" reason="Adjacent"/>
+  <disable_collisions link1="${prefix}gripper_base_link" link2="${prefix}gripper_left_link" reason="Adjacent"/>
+  <disable_collisions link1="${prefix}gripper_base_link" link2="${prefix}gripper_right_link" reason="Adjacent"/>
+  <disable_collisions link1="${prefix}gripper_left_link" link2="${prefix}gripper_left_finger" reason="Adjacent"/>
+  <disable_collisions link1="${prefix}gripper_right_link" link2="${prefix}gripper_right_finger" reason="Adjacent"/>
 </robot>

File: src/vendor_robot_simulation/urdf/g4_mobile_depth.gazebo.urdf.xacro (robot description, xacro)
@@ -18,8 +18,16 @@
     </gazebo>
   </xacro:macro>
-  <xacro:arm_gazebo_properties link_name="base_link"/><xacro:arm_gazebo_properties link_name="Link1"/>
-  <xacro:arm_gazebo_properties link_name="Link2"/><xacro:arm_gazebo_properties link_name="Link3"/>
-  <xacro:arm_gazebo_properties link_name="Link4"/><xacro:arm_gazebo_properties link_name="Link5"/>
+  <xacro:arm_gazebo_properties link_name="base_link"/>
+  <xacro:arm_gazebo_properties link_name="Link1"/>
+  <xacro:arm_gazebo_properties link_name="Link2"/>
+  <xacro:arm_gazebo_properties link_name="Link3"/>
+  <xacro:arm_gazebo_properties link_name="Link4"/>
+  <xacro:arm_gazebo_properties link_name="Link5"/>
   <xacro:arm_gazebo_properties link_name="Link6"/>
+  <xacro:arm_gazebo_properties link_name="gripper_base_link"/>
+  <xacro:arm_gazebo_properties link_name="gripper_left_link"/>
+  <xacro:arm_gazebo_properties link_name="gripper_right_link"/>
+  <xacro:arm_gazebo_properties link_name="gripper_left_finger"/>
+  <xacro:arm_gazebo_properties link_name="gripper_right_finger"/>
   <ros2_control name="${prefix}GazeboSystem" type="system">
     <hardware><plugin>gazebo_ros2_control/GazeboSystem</plugin></hardware>
@@ -31,7 +39,33 @@
       </joint>
     </xacro:macro>
-    <xacro:arm_joint_interface joint_name="joint1"/><xacro:arm_joint_interface joint_name="joint2"/>
-    <xacro:arm_joint_interface joint_name="joint3"/><xacro:arm_joint_interface joint_name="joint4"/>
-    <xacro:arm_joint_interface joint_name="joint5"/><xacro:arm_joint_interface joint_name="joint6"/>
+    <xacro:arm_joint_interface joint_name="joint1"/>
+    <xacro:arm_joint_interface joint_name="joint2"/>
+    <xacro:arm_joint_interface joint_name="joint3"/>
+    <xacro:arm_joint_interface joint_name="joint4"/>
+    <xacro:arm_joint_interface joint_name="joint5"/>
+    <xacro:arm_joint_interface joint_name="joint6"/>
+    <!-- The model owns the mimic declaration; Gazebo owns the actuator interface. -->
+    <joint name="${prefix}gripper_left_joint">
+      <command_interface name="position"/>
+      <state_interface name="position"><param name="initial_value">-0.055</param></state_interface>
+      <state_interface name="velocity"/>
+    </joint>
+    <joint name="${prefix}gripper_right_joint">
+      <param name="mimic">${prefix}gripper_left_joint</param>
+      <param name="multiplier">-1</param>
+      <!-- Mimic joints are state-only: gripper_left_joint is the sole actuator. -->
+      <state_interface name="position"/><state_interface name="velocity"/>
+    </joint>
+    <!-- The diff-drive Gazebo plugin commands these wheels.  ros2_control only
+         exports their state so robot_state_publisher and MoveIt see a complete
+         model state. -->
+    <joint name="${prefix}left_wheel_joint">
+      <state_interface name="position"/>
+      <state_interface name="velocity"/>
+    </joint>
+    <joint name="${prefix}right_wheel_joint">
+      <state_interface name="position"/>
+      <state_interface name="velocity"/>
+    </joint>
   </ros2_control>
   <gazebo>
@@ -92,5 +126,5 @@
     <parent link="${prefix}Link6"/>
     <child link="${prefix}depth_camera_link"/>
-    <origin xyz="0.08 0 0" rpy="0 0 0"/>
+    <origin xyz="0.08 0 -0.03" rpy="0 0 0"/>
   </joint>
   <link name="${prefix}depth_camera_optical_frame"/>
@@ -99,5 +133,5 @@
     <child link="${prefix}depth_camera_optical_frame"/>
     <!-- ROS optical frame: X right, Y down, Z forward. -->
-    <origin xyz="0 0 0" rpy="-1.57079632679 0 -1.57079632679"/>
+    <origin xyz="0.08 0 0" rpy="-1.57079632679 0 -1.57079632679"/>
   </joint>
   <gazebo reference="${prefix}depth_camera_link">
@@ -121,5 +155,8 @@
       <max_wheel_torque>20.0</max_wheel_torque><max_wheel_acceleration>4.0</max_wheel_acceleration>
       <publish_odom>true</publish_odom><publish_odom_tf>true</publish_odom_tf><publish_wheel_tf>true</publish_wheel_tf>
-      <odometry_frame>odom</odometry_frame><robot_base_frame>${prefix}mobile_base_link</robot_base_frame>
+      <!-- Publish odom -> base_footprint.  The URDF then contributes the
+           fixed base_footprint -> mobile_base_link transform, yielding one
+           connected TF tree (rather than two parents for mobile_base_link). -->
+      <odometry_frame>odom</odometry_frame><robot_base_frame>${prefix}base_footprint</robot_base_frame>
     </plugin>
   </gazebo>
