Commit message: update-8.28

File: src/vendor_robot_description/urdf/gripper.xacro (robot description, xacro)
@@ -123,4 +123,22 @@
       </collision>
     </link>
+    <!--
+      夹爪实际夹持中心。手指碰撞网格在 gripper_base_link 的本地 Z 方向
+      覆盖 0.0805–0.1535 m，中心约为 0.117 m。MTC 以此 Link 作为 IK
+      坐标系，使物块中心落在两指的有效夹持区，而非停在手指上方。
+    -->
+    <link name="${prefix}gripper_tcp"/>
+    <joint
+        name="${prefix}gripper_tcp_joint"
+        type="fixed">
+        <parent
+            link="${prefix}gripper_base_link"/>
+        <child
+            link="${prefix}gripper_tcp"/>
+        <!-- 该偏置已由手指网格尺寸校准；修改后需同步检查 MTC 抓取效果。 -->
+        <origin
+            xyz="0 0 0.13"
+            rpy="0 0 0"/>
+    </joint>
   </xacro:macro>
 </robot>

File: src/vendor_robot_moveit_config/config/G4.srdf.xacro (robot description, xacro)
@@ -35,8 +35,9 @@
     <joint name="${prefix}gripper_left_joint" value="-0.0027"/>
   </group_state>
-  <!-- About 54 mm jaw spacing: suitable for the 50 mm gazebo_grasp_box.
-       "closed" remains the empty-gripper, fully closed state. -->
+  <!-- -0.0275 对应约 49 mm 的指间距，比 50 mm 方块小约 1 mm，
+       用于在规划中模拟夹持接触；MTC 会显式允许手指与目标碰撞。
+       closed 保留为空载时两指几乎相合的状态。 -->
   <group_state name="grasp" group="gripper">
-    <joint name="${prefix}gripper_left_joint" value="-0.029"/>
+    <joint name="${prefix}gripper_left_joint" value="-0.0275"/>
   </group_state>
   <disable_collisions link1="${prefix}Link1" link2="${prefix}Link2" reason="Adjacent"/>

File: src/vendor_robot_simulation/urdf/g4_mobile_depth.gazebo.urdf.xacro (robot description, xacro)
@@ -3,5 +3,7 @@
 <robot xmlns:xacro="http://www.ros.org/wiki/xacro" name="g4_mobile_depth">
   <xacro:arg name="prefix" default=""/>
-  <xacro:arg name="use_gravity" default="true"/>
+  <xacro:arg name="use_gravity" default="false"/>
+  <!-- true：底盘固定在世界坐标系；false：为恢复差速移动预留。 -->
+  <xacro:arg name="fixed_mobile_base" default="true"/>
   <xacro:arg name="initial_positions_file" default="$(find vendor_robot_description)/config/initial_positions.yaml"/>
   <xacro:arg name="controllers_file" default="$(find vendor_robot_simulation)/config/controllers.yaml"/>
@@ -57,7 +59,6 @@
       <state_interface name="position"/><state_interface name="velocity"/>
     </joint>
-    <!-- The diff-drive Gazebo plugin commands these wheels.  ros2_control only
-         exports their state so robot_state_publisher and MoveIt see a complete
-         model state. -->
+    <!-- 当前移动底盘固定在世界坐标系中；轮子只导出状态，保证
+         robot_state_publisher 与 MoveIt 获得完整的机器人关节状态。 -->
     <joint name="${prefix}left_wheel_joint">
       <state_interface name="position"/>
@@ -83,4 +84,5 @@
     </plugin>
   </gazebo>
+  <!-- 左右两差速轮设置和joint设置在mobile_base_link上. -->
   <xacro:macro name="wheel" params="name y">
     <link name="${prefix}${name}">
@@ -97,10 +99,9 @@
       <child link="${prefix}${name}"/>
       <!-- mobile_base_link is elevated; keep wheel contact at world z=0. -->
-      <origin xyz="0 ${y} ${wheel_radius / 2.0}" rpy="0 0 0"/>
+      <origin xyz="0.15 ${y} ${wheel_radius / 2.0}" rpy="0 0 0"/>
       <axis xyz="0 1 0"/>
     </joint>
   </xacro:macro>
-  <!-- A massless root prevents KDL/robot_state_publisher from discarding the
-       mobile-base inertia. Gazebo's odom TF targets mobile_base_link. -->
+  <!-- 移动底盘的size设置. -->
   <link name="${prefix}base_footprint"/>
   <link name="${prefix}mobile_base_link">
@@ -113,4 +114,17 @@
     <collision><origin xyz="0 0 0.10"/><geometry><box size="0.70 0.52 0.20"/></geometry></collision>
   </link>
+  <!--
+    将移动底盘固定到 Gazebo 世界坐标系。
+    这样开启重力后，底盘和三个轮子不会因轮地接触、惯量或残余速度而移动；
+    机械臂的各个可动关节仍由 ros2_control 正常驱动。
+  -->
+  <xacro:if value="$(arg fixed_mobile_base)">
+    <link name="world"/>
+    <joint name="${prefix}world_to_mobile_base" type="fixed">
+      <parent link="world"/>
+      <child link="${prefix}mobile_base_link"/>
+      <origin xyz="0 0 0" rpy="0 0 0"/>
+    </joint>
+  </xacro:if>
   <joint name="${prefix}mobile_base_to_base_footprint" type="fixed">
     <parent link="${prefix}mobile_base_link"/><child link="${prefix}base_footprint"/>
@@ -171,5 +185,5 @@
     <gravity>$(arg use_gravity)</gravity>
     <sensor name="depth_camera_sensor" type="depth">
-      <always_on>true</always_on><update_rate>30</update_rate><visualize>false</visualize>
+      <always_on>true</always_on><update_rate>10</update_rate><visualize>false</visualize>
       <camera><horizontal_fov>1.047</horizontal_fov><image><width>640</width><height>480</height><format>B8G8R8</format></image><depth_camera/><clip><near>0.10</near><far>8.0</far></clip></camera>
       <plugin name="depth_camera_controller" filename="libgazebo_ros_camera.so">
@@ -181,4 +195,8 @@
     </sensor>
   </gazebo>
+  <!--
+    差速驱动配置暂时保留但不加载。移动底盘固定时若加载该插件，插件仍会
+    向左右轮施加速度命令，可能引发轮地接触的不稳定。需要恢复小车移动时，
+    将启动参数 fixed_mobile_base 设为 false，并取消下面整段注释。
   <gazebo>
     <plugin name="mobile_base_diff_drive" filename="libgazebo_ros_diff_drive.so">
@@ -189,9 +207,7 @@
       <max_wheel_torque>20.0</max_wheel_torque><max_wheel_acceleration>4.0</max_wheel_acceleration>
       <publish_odom>true</publish_odom><publish_odom_tf>true</publish_odom_tf><publish_wheel_tf>true</publish_wheel_tf>
-      <!-- Publish odom -> base_footprint.  The URDF then contributes the
-           fixed base_footprint -> mobile_base_link transform, yielding one
-           connected TF tree (rather than two parents for mobile_base_link). -->
       <odometry_frame>odom</odometry_frame><robot_base_frame>${prefix}mobile_base_link</robot_base_frame>
     </plugin>
   </gazebo>
+  -->
 </robot>
