Commit message: 更新

File: src/vendor_robot_moveit_config/config/G4.srdf.xacro (robot description, xacro)
@@ -1,4 +1,5 @@
 <?xml version="1.0" encoding="UTF-8"?>
-<robot xmlns:xacro="http://www.ros.org/wiki/xacro" name="G4">
+<robot xmlns:xacro="http://www.ros.org/wiki/xacro" name="$(arg robot_name)">
+  <xacro:arg name="robot_name" default="G4"/>
   <xacro:arg name="prefix" default=""/>
   <xacro:property name="prefix" value="$(arg prefix)"/>

File: src/vendor_robot_simulation/urdf/g4_mobile_depth.gazebo.urdf.xacro (robot description, xacro)
@@ -48,5 +48,5 @@
     <joint name="${prefix}gripper_left_joint">
       <command_interface name="position"/>
-      <state_interface name="position"><param name="initial_value">-0.055</param></state_interface>
+      <state_interface name="position"><param name="initial_value">${initial_positions['gripper_left_joint']}</param></state_interface>
       <state_interface name="velocity"/>
     </joint>
@@ -65,4 +65,12 @@
     </joint>
     <joint name="${prefix}right_wheel_joint">
+      <state_interface name="position"/>
+      <state_interface name="velocity"/>
+    </joint>
+    <joint name="${prefix}caster_swivel_joint">
+      <state_interface name="position"/>
+      <state_interface name="velocity"/>
+    </joint>
+    <joint name="${prefix}caster_wheel_joint">
       <state_interface name="position"/>
       <state_interface name="velocity"/>
@@ -88,5 +96,6 @@
       <parent link="${prefix}mobile_base_link"/>
       <child link="${prefix}${name}"/>
-      <origin xyz="0 ${y} ${wheel_radius}" rpy="0 0 0"/>
+      <!-- mobile_base_link is elevated; keep wheel contact at world z=0. -->
+      <origin xyz="0 ${y} ${wheel_radius / 2.0}" rpy="0 0 0"/>
       <axis xyz="0 1 0"/>
     </joint>
@@ -95,8 +104,4 @@
        mobile-base inertia. Gazebo's odom TF targets mobile_base_link. -->
   <link name="${prefix}base_footprint"/>
-  <joint name="${prefix}base_footprint_to_mobile_base" type="fixed">
-    <parent link="${prefix}base_footprint"/><child link="${prefix}mobile_base_link"/>
-    <origin xyz="0 0 0" rpy="0 0 0"/>
-  </joint>
   <link name="${prefix}mobile_base_link">
     <inertial>
@@ -108,7 +113,28 @@
     <collision><origin xyz="0 0 0.10"/><geometry><box size="0.70 0.52 0.20"/></geometry></collision>
   </link>
+  <joint name="${prefix}mobile_base_to_base_footprint" type="fixed">
+    <parent link="${prefix}mobile_base_link"/><child link="${prefix}base_footprint"/>
+    <origin xyz="0 0 -0.05" rpy="0 0 0"/>
+  </joint>
   <gazebo reference="${prefix}mobile_base_link"><material>Gazebo/Blue</material><gravity>$(arg use_gravity)</gravity></gazebo>
   <xacro:wheel name="left_wheel" y="${wheel_separation / 2.0}"/>
   <xacro:wheel name="right_wheel" y="${-wheel_separation / 2.0}"/>
+  <!-- Rear swivel caster supporting the elevated chassis. -->
+  <link name="${prefix}caster_swivel_link">
+    <inertial><mass value="0.15"/><inertia ixx="0.0002" ixy="0" ixz="0" iyy="0.0002" iyz="0" izz="0.0002"/></inertial>
+  </link>
+  <joint name="${prefix}caster_swivel_joint" type="continuous">
+    <parent link="${prefix}mobile_base_link"/><child link="${prefix}caster_swivel_link"/>
+    <origin xyz="-0.28 0 0" rpy="0 0 0"/><axis xyz="0 0 1"/>
+  </joint>
+  <link name="${prefix}caster_wheel">
+    <inertial><mass value="0.4"/><inertia ixx="0.001" ixy="0" ixz="0" iyy="0.001" iyz="0" izz="0.001"/></inertial>
+    <visual><origin rpy="1.57079632679 0 0"/><geometry><cylinder radius="0.06" length="0.04"/></geometry><material name="caster_black"><color rgba="0.03 0.03 0.03 1"/></material></visual>
+    <collision><origin rpy="1.57079632679 0 0"/><geometry><cylinder radius="0.06" length="0.04"/></geometry></collision>
+  </link>
+  <joint name="${prefix}caster_wheel_joint" type="continuous">
+    <parent link="${prefix}caster_swivel_link"/><child link="${prefix}caster_wheel"/>
+    <origin xyz="0 0 0.01" rpy="0 0 0"/><axis xyz="0 1 0"/>
+  </joint>
   <!-- The arm model's root is base -> base_link. Mount base above the chassis. -->
   <joint name="${prefix}mobile_base_to_robot_base" type="fixed">
@@ -158,5 +184,5 @@
            fixed base_footprint -> mobile_base_link transform, yielding one
            connected TF tree (rather than two parents for mobile_base_link). -->
-      <odometry_frame>odom</odometry_frame><robot_base_frame>${prefix}base_footprint</robot_base_frame>
+      <odometry_frame>odom</odometry_frame><robot_base_frame>${prefix}mobile_base_link</robot_base_frame>
     </plugin>
   </gazebo>

Commit message: update

File: src/vendor_robot_moveit_config/config/G4.srdf.xacro (robot description, xacro)
@@ -29,8 +29,14 @@
   </group_state>
   <group_state name="open" group="gripper">
-    <joint name="${prefix}gripper_left_joint" value="-0.055"/>
+    <!-- Match gazebo_ros2_control's initial gripper_left_joint state. -->
+    <joint name="${prefix}gripper_left_joint" value="-0.054"/>
   </group_state>
   <group_state name="closed" group="gripper">
     <joint name="${prefix}gripper_left_joint" value="-0.0027"/>
+  </group_state>
+  <!-- About 54 mm jaw spacing: suitable for the 50 mm gazebo_grasp_box.
+       "closed" remains the empty-gripper, fully closed state. -->
+  <group_state name="grasp" group="gripper">
+    <joint name="${prefix}gripper_left_joint" value="-0.029"/>
   </group_state>
   <disable_collisions link1="${prefix}Link1" link2="${prefix}Link2" reason="Adjacent"/>
@@ -50,3 +56,11 @@
   <disable_collisions link1="${prefix}gripper_left_link" link2="${prefix}gripper_left_finger" reason="Adjacent"/>
   <disable_collisions link1="${prefix}gripper_right_link" link2="${prefix}gripper_right_finger" reason="Adjacent"/>
+  <!-- The mobile chassis, mounted arm base, and support wheels deliberately
+       overlap in the simplified collision geometry. They are mechanically
+       connected links, so treating these pairs as self-collisions invalidates
+       every MTC grasp candidate before gripper-object contact is allowed. -->
+  <disable_collisions link1="${prefix}mobile_base_link" link2="${prefix}base_link" reason="Adjacent"/>
+  <disable_collisions link1="${prefix}mobile_base_link" link2="${prefix}left_wheel" reason="Adjacent"/>
+  <disable_collisions link1="${prefix}mobile_base_link" link2="${prefix}right_wheel" reason="Adjacent"/>
+  <disable_collisions link1="${prefix}mobile_base_link" link2="${prefix}caster_wheel" reason="Adjacent"/>
 </robot>

File: src/vendor_robot_simulation/urdf/g4_mobile_depth.gazebo.urdf.xacro (robot description, xacro)
@@ -120,4 +120,9 @@
   <xacro:wheel name="left_wheel" y="${wheel_separation / 2.0}"/>
   <xacro:wheel name="right_wheel" y="${-wheel_separation / 2.0}"/>
+  <!-- Keep all mobile-base links governed by the launch use_gravity argument.
+       Without these overrides the wheels inherit world gravity even when the
+       rest of the robot is configured with use_gravity:=false. -->
+  <gazebo reference="${prefix}left_wheel"><gravity>$(arg use_gravity)</gravity></gazebo>
+  <gazebo reference="${prefix}right_wheel"><gravity>$(arg use_gravity)</gravity></gazebo>
   <!-- Rear swivel caster supporting the elevated chassis. -->
   <link name="${prefix}caster_swivel_link">
@@ -137,4 +142,6 @@
     <origin xyz="0 0 0.01" rpy="0 0 0"/><axis xyz="0 1 0"/>
   </joint>
+  <gazebo reference="${prefix}caster_swivel_link"><gravity>$(arg use_gravity)</gravity></gazebo>
+  <gazebo reference="${prefix}caster_wheel"><gravity>$(arg use_gravity)</gravity></gazebo>
   <!-- The arm model's root is base -> base_link. Mount base above the chassis. -->
   <joint name="${prefix}mobile_base_to_robot_base" type="fixed">
@@ -162,4 +169,5 @@
   </joint>
   <gazebo reference="${prefix}depth_camera_link">
+    <gravity>$(arg use_gravity)</gravity>
     <sensor name="depth_camera_sensor" type="depth">
       <always_on>true</always_on><update_rate>30</update_rate><visualize>false</visualize>

Commit message: update-9.3

File: src/vendor_robot_moveit_config/config/G4.srdf.xacro (robot description, xacro)
@@ -39,5 +39,5 @@
        closed 保留为空载时两指几乎相合的状态。 -->
   <group_state name="grasp" group="gripper">
-    <joint name="${prefix}gripper_left_joint" value="-0.0275"/>
+    <joint name="${prefix}gripper_left_joint" value="-0.027"/>
   </group_state>
   <disable_collisions link1="${prefix}Link1" link2="${prefix}Link2" reason="Adjacent"/>

File: src/vendor_robot_simulation/urdf/g4_mobile_depth.gazebo.urdf.xacro (robot description, xacro)
@@ -6,4 +6,6 @@
   <!-- true：底盘固定在世界坐标系；false：为恢复差速移动预留。 -->
   <xacro:arg name="fixed_mobile_base" default="true"/>
+  <!-- 机器人相对于世界坐标系的初始高度；由 URDF TF 统一表达。 -->
+  <xacro:arg name="spawn_z" default="0.055"/>
   <xacro:arg name="initial_positions_file" default="$(find vendor_robot_description)/config/initial_positions.yaml"/>
   <xacro:arg name="controllers_file" default="$(find vendor_robot_simulation)/config/controllers.yaml"/>
@@ -124,5 +126,5 @@
       <parent link="world"/>
       <child link="${prefix}mobile_base_link"/>
-      <origin xyz="0 0 0" rpy="0 0 0"/>
+      <origin xyz="0 0 $(arg spawn_z)" rpy="0 0 0"/>
     </joint>
   </xacro:if>
@@ -180,5 +182,5 @@
     <child link="${prefix}depth_camera_optical_frame"/>
     <!-- ROS optical frame: X right, Y down, Z forward. -->
-    <origin xyz="0.08 0 0" rpy="-1.57079632679 0 -1.57079632679"/>
+    <origin xyz="0.0 0 0" rpy="-1.57079632679 0 -1.57079632679"/>
   </joint>
   <gazebo reference="${prefix}depth_camera_link">

Commit message: update-9.4

File: src/vendor_robot_moveit_config/config/G4.srdf.xacro (robot description, xacro)
@@ -39,5 +39,5 @@
        closed 保留为空载时两指几乎相合的状态。 -->
   <group_state name="grasp" group="gripper">
-    <joint name="${prefix}gripper_left_joint" value="-0.027"/>
+    <joint name="${prefix}gripper_left_joint" value="-0.026"/>
   </group_state>
   <disable_collisions link1="${prefix}Link1" link2="${prefix}Link2" reason="Adjacent"/>
